File: board/board.kicad_pcb (KiCad board)
At the start: 2 copper layers, 45 x 29 mm, 19 parts, among them J1 014_PoE_controlled, J2 003_power, U1 BD9G341AEFJ-E2

Commit message: added lcsc part numbers
Connections:
- net Net-(C5-Pad1) renamed /step-down/SW
- net Net-(C5-Pad2) renamed /step-down/BST
- net Net-(C6-Pad1) renamed /step-down/VCC
- net Net-(R5-Pad2) renamed /step-down/FB
